File: Component tester/Component tester.kicad_pcb (KiCad board)
At the start: 2 copper layers, 38.6 x 43 mm, 8 parts, among them J2 Conn_01x02, J3 Conn_01x04, J4 Conn_01x04, U2 Seeeduino Xiao rp2040

Commit message: Finished PCB
Parts:
- added SW1: SW_Push, Button_Switch_THT:SW_PUSH_6mm, F.Cu at (124.0, 48.0)
- added SW2: SW_Push, Button_Switch_THT:SW_PUSH_6mm, F.Cu at (124.0, 58.0)
- moved R3 11.0 mm to (123.0, 40.0)
- moved J2 11.0 mm to (127.0, 40.0)
- moved R4 10.5 mm to (123.0, 44.0)
- moved R1 7.49 mm to (120.0, 30.9)
- moved R2 7.49 mm to (120.0, 34.9)
Connections:
- U2 pad 3: unconnected-(U2-P28-Pad3)_1 -> SW1
- U2 pad 4: unconnected-(U2-P29-Pad4)_1 -> SW2
Routing:
- net SW1: track 0.00 -> 32.1 mm
- net SW2: track 0.00 -> 25.7 mm
- net IN_5V_DIV: track 37.4 -> 42.2 mm
- net Continuity: track 28.8 -> 33.4 mm
- net GND: track 0.00 -> 1.30 mm
- net IN_5V: track 8.85 -> 8.09 mm
- added copper zone on B.Cu, net GND
- added copper zone on F.Cu, net GND
Other:
- board size 38.6 x 43 mm -> 38.6 x 43.6 mm
- board text added: "Menu"
- board text added: "Select"
- board text removed: "XIAO"
