File: Component tester/Component tester.kicad_sch (KiCad schematic)
At the start: 8 parts, among them J2 Conn_01x02, J3 Conn_01x04, J4 Conn_01x04, U2 Seeeduino Xiao rp2040

Commit message: Finished PCB
Parts:
- added SW1, SW2: SW_Push, Button_Switch_THT:SW_PUSH_6mm, symbol Switch:SW_Push
Connections:
- net GND: now also SW1.2, SW2.2
- net SW1: now reaches U2.3 (P28)
- net SW1: now also SW1.1
- net SW2: now reaches U2.4 (P29)
- net SW2: now also SW2.1
- no-connect marks 13 -> 11
